File: hardware/NORMMotorControlBoard.kicad_pcb (KiCad board)
At the start: 2 copper layers, 75 x 160 mm, 32 parts, among them J1 Front Right Motor, J2 Front Left Motor, J3 Back Right Motor, J4 Back Left Motor, J5 Conn_01x02_Socket, J6 SparePins, J7 SparePins, SW1 Reset, U1 Front Driver, U2 Back Driver, U3 74HC595

Commit message: V1.3
Parts:
- removed J7: SparePins, Connector_PinHeader_2.54mm:PinHeader_1x05_P2.54mm_Vertical
- J6: footprint Connector_PinHeader_2.54mm:PinHeader_1x05_P2.54mm_Horizontal -> Connector_PinHeader_2.54mm:PinHeader_1x08_P2.54mm_Horizontal
- moved J6 5.64 mm to (227.6, 274.8)
- moved U3 3.43 mm to (264.2, 222.2)
- moved A1 0.87 mm to (218.7, 212.7)
Connections:
- A1 pad 10: FL_ENC_SEC -> BR_ENC_PRI
- A1 pad 11: FR_ENC_PRI -> BL_ENC_PRI
- A1 pad 12: FR_ENC_SEC -> BR_SPEED
- A1 pad 13: BL_ENC_PRI -> D10
- A1 pad 14: BL_ENC_SEC -> D11
- A1 pad 19: SR_DATA -> SR_CLOCK
- A1 pad 21: SR_CLOCK -> SR_DATA
- A1 pad 22: A3 -> BL_ENC_SEC
- A1 pad 23: A4 -> FL_ENC_SEC
- A1 pad 24: A5 -> FR_ENC_SEC
- A1 pad 25: BR_ENC_PRI -> BR_ENC_SEC
- A1 pad 26: BR_ENC_SEC -> A7
- A1 pad 5: FL_SPEED -> FL_ENC_PRI
- A1 pad 6: FR_SPEED -> FL_SPEED
- A1 pad 7: BL_SPEED -> FR_ENC_PRI
- A1 pad 8: BR_SPEED -> FR_SPEED
- A1 pad 9: FL_ENC_PRI -> BL_SPEED
- J6 pad 1: +3.3V -> A7
- J6 pad 2: GND -> D13
- J6 pad 3: A3 -> D12
- J6 pad 4: A4 -> D11
- J6 pad 5: A5 -> D10
Routing:
- net +3.3V: track 0.00 -> 363.5 mm, vias 0 -> 1
- net +5V: track 0.00 -> 179.7 mm
- net FL_ENC_SEC: track 0.00 -> 159.9 mm, vias 0 -> 1
- net FL_ENC_PRI: track 0.00 -> 144.9 mm
- net FR_ENC_SEC: track 0.00 -> 123.0 mm, vias 0 -> 1
- net +12V: track 0.00 -> 117.4 mm
- net FR_ENC_PRI: track 0.00 -> 111.2 mm, vias 0 -> 1
- net BL_ENC_PRI: track 0.00 -> 103.2 mm, vias 0 -> 1
- net Net-(A1-~{RESET}-Pad3): track 0.00 -> 98.0 mm
- net BL_ENC_SEC: track 0.00 -> 93.8 mm
- net FL_SPEED: track 0.00 -> 92.8 mm
- net FR_SPEED: track 0.00 -> 85.3 mm
- net BR_ENC_PRI: track 0.00 -> 59.5 mm, vias 0 -> 1
- net BR_ENC_SEC: track 0.00 -> 57.6 mm
- net A7: track 0.00 -> 57.1 mm
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Other:
- board text added: "A7"
- board text added: "D10"
- board text added: "D11"
- board text removed: "3.3V"
- board text removed: "A3"
- board text removed: "A4"
- board text removed: "A5"
